Commit message: Move project from GitLab to GitHub

File: momo_description/urdf/momo_description.urdf (robot description, URDF)
Before this commit: robot momo_description, 6 links, 5 joints
Links:
- added link back_logitech, mass 0.0873967458266511; collision mesh filename=package://momo_description/meshes/visual/back_logitech.STL; visual mesh filename=package://momo_description/meshes/visual/back_logitech.STL
- added link front_logitech, mass 0.0873967458266508; collision mesh filename=package://momo_description/meshes/visual/front_logitech.STL; visual mesh filename=package://momo_description/meshes/visual/front_logitech.STL
- added link ifm_camera, mass 0.0711675681323896; collision mesh filename=package://momo_description/meshes/visual/ifm_camera.STL; visual mesh filename=package://momo_description/meshes/visual/ifm_camera.STL
- added link left_logitech, mass 0.0873967458266511; collision mesh filename=package://momo_description/meshes/visual/left_logitech.STL; visual mesh filename=package://momo_description/meshes/visual/left_logitech.STL
- added link lidar, mass 0.605610123538718; collision mesh filename=package://momo_description/meshes/visual/lidar.STL; visual mesh filename=package://momo_description/meshes/visual/lidar.STL
- added link realsense_d435i, mass 0.0457663452618203; collision mesh filename=package://momo_description/meshes/visual/realsense_d435i.STL; visual mesh filename=package://momo_description/meshes/visual/realsense_d435i.STL
- added link realsense_t265, mass 0.0311240910368595; collision mesh filename=package://momo_description/meshes/visual/realsense_t265.STL; visual mesh filename=package://momo_description/meshes/visual/realsense_t265.STL
- added link right_logitech, mass 0.0873967458266508; collision mesh filename=package://momo_description/meshes/visual/right_logitech.STL; visual mesh filename=package://momo_description/meshes/visual/right_logitech.STL
- link back_right_wheel: mass 0.852354640622837 -> 0.852354640622838
- link base_link: mass 5.93891084584059 -> 9.12874381762573
- link front_left_wheel: mass 0.852354640622835 -> 0.852354640622848
- link front_right_wheel: mass 0.85235460510222 -> 0.852354605102217
Joints:
- added joint back_logitech_joint: type fixed, parent base_link, child back_logitech, origin xyz=-0.254567242746362 0.0415958603547848 0.418952968841513 rpy=-1.5707963267949 0 1.5707963267949, axis 0 0 0
- added joint front_logitech_joint: type fixed, parent base_link, child front_logitech, origin xyz=0.154732757253638 0.0412775530270625 0.418952968841513 rpy=-1.5707963267949 0 -1.5707963267949, axis 0 0 0
- added joint ifm_camera_joint: type fixed, parent base_link, child ifm_camera, origin xyz=0.30569 0.014587 0.26684 rpy=-1.5708 0 -1.5708, axis 0 0 0
- added joint left_logitech_joint: type fixed, parent base_link, child left_logitech, origin xyz=-0.00225808908250899 0.248086706690936 0.418952968841515 rpy=-1.5707963267949 0 0, axis 0 0 0
- added joint lidar_joint: type fixed, parent base_link, child lidar, origin xyz=-0.00241706738442254 0.0414368820528667 0.478357617954853 rpy=0 0 -1.5707963267949, axis 0 0 0
- added joint realsense_d435i_joint: type fixed, parent base_link, child realsense_d435i, origin xyz=-0.404814742746363 0.0344707026853986 0.279039270865987 rpy=-1.5707963267949 0 1.5707963267949, axis 0 0 0
- added joint realsense_t265_joint: type fixed, parent base_link, child realsense_t265, origin xyz=0.184822757253643 0.0443427066909039 0.337457617954855 rpy=-1.5707963267949 0 -1.5707963267949, axis 0 0 0
- added joint right_logitech_joint: type fixed, parent base_link, child right_logitech, origin xyz=-0.00257639641022331 -0.165213293309076 0.418952968841513 rpy=-1.5707963267949 0 3.14159265358979, axis 0 0 0
- joint back_left_wheel_joint: origin xyz=-0.2735 0.318 0.059993 rpy=1.5708 0 0 -> xyz=-0.273501168246142 0.318000000000003 0.0599931160727954 rpy=1.5707963267949 0 0
- joint back_right_wheel_joint: origin xyz=-0.27349 -0.318 0.059998 rpy=1.5708 0 0 -> xyz=-0.27349334578749 -0.318000000000002 0.0599978846492716 rpy=1.5707963267949 0 0
- joint front_left_wheel_joint: origin xyz=0.26849 0.318 0.059999 rpy=1.5708 0 0 -> xyz=0.268493050220139 0.317999999999998 0.0599993263438537 rpy=1.5707963267949 0 0
