Commit message: Add remaining camera plugins for gazebo

File: momo_description/urdf/camera_plugin.xacro (robot description, xacro)
@@ -18,8 +18,74 @@
                     </clip>
                 </camera>
-                <plugin name="camera_controller" filename="libgazebo_ros_camera.so">
+                <plugin name="front_camera_controller" filename="libgazebo_ros_camera.so">
                 <frame_name>front_logitech_optical</frame_name>
             </plugin>
         </sensor>
     </gazebo>
+    <gazebo reference="right_logitech">
+        <sensor name="right_logitech_camera" type="camera">
+            <pose> 0 0 0 0 0 0 </pose>
+            <visualize>true</visualize>
+            <update_rate>10</update_rate>
+                <camera>
+                    <horizontal_fov>1.089</horizontal_fov>
+                    <image>
+                        <format>R8G8B8</format>
+                        <width>640</width>
+                        <height>480</height>
+                    </image>
+                    <clip>
+                        <near>0.05</near>
+                        <far>8.0</far>
+                    </clip>
+                </camera>
+                <plugin name="right_camera_controller" filename="libgazebo_ros_camera.so">
+                <frame_name>right_logitech_optical</frame_name>
+            </plugin>
+        </sensor>
+    </gazebo>
+    <gazebo reference="back_logitech">
+        <sensor name="back_logitech_camera" type="camera">
+            <pose> 0 0 0 0 0 0 </pose>
+            <visualize>true</visualize>
+            <update_rate>10</update_rate>
+                <camera>
+                    <horizontal_fov>1.089</horizontal_fov>
+                    <image>
+                        <format>R8G8B8</format>
+                        <width>640</width>
+                        <height>480</height>
+                    </image>
+                    <clip>
+                        <near>0.05</near>
+                        <far>8.0</far>
+                    </clip>
+                </camera>
+                <plugin name="back_camera_controller" filename="libgazebo_ros_camera.so">
+                <frame_name>back_logitech_optical</frame_name>
+            </plugin>
+        </sensor>
+    </gazebo>
+    <gazebo reference="left_logitech">
+        <sensor name="left_logitech_camera" type="camera">
+            <pose> 0 0 0 0 0 0 </pose>
+            <visualize>true</visualize>
+            <update_rate>10</update_rate>
+                <camera>
+                    <horizontal_fov>1.089</horizontal_fov>
+                    <image>
+                        <format>R8G8B8</format>
+                        <width>640</width>
+                        <height>480</height>
+                    </image>
+                    <clip>
+                        <near>0.05</near>
+                        <far>8.0</far>
+                    </clip>
+                </camera>
+                <plugin name="left_camera_controller" filename="libgazebo_ros_camera.so">
+                <frame_name>left_logitech_optical</frame_name>
+            </plugin>
+        </sensor>
+    </gazebo>
 </robot>

File: momo_description/urdf/momo_perception_module.xacro (robot description, xacro)
@@ -10,5 +10,5 @@
         </inertial>
         <visual>
-            <origin xyz="0 0 0" rpy="0 0 0" />
+            <origin xyz="0 0 0" rpy="-1.57 0 -1.57" />
             <geometry>
                 <mesh filename="file://$(find momo_description)/meshes/visual/front_logitech.STL" />
@@ -19,5 +19,5 @@
         </visual>
         <collision>
-            <origin xyz="0 0 0" rpy="0 0 0" />
+            <origin xyz="0 0 0" rpy="-1.57 0 -1.57" />
             <geometry>
                 <mesh filename="file://$(find momo_description)/meshes/visual/front_logitech.STL" />
@@ -29,4 +29,5 @@
     </gazebo>
     <joint name="front_logitech_joint" type="fixed">
+        <!-- <origin xyz="0.154732757253638 0.0412775530270625 0.418952968841513" rpy="-1.5707963267949 0 -1.5707963267949" /> -->
         <origin xyz="0.154732757253638 0.0412775530270625 0.418952968841513" rpy="0 0 0" />
         <parent link="base_link" />
@@ -34,6 +35,6 @@
         <axis xyz="0 0 0" />
     </joint>
-    <!-- for camera plugin -->
     <joint name="front_logitech_optical_joint" type="fixed">
+        <!-- <origin xyz="0.154732757253638 0.0412775530270625 0.418952968841513" rpy="-1.5707963267949 0 -1.5707963267949" /> -->
         <origin xyz="0 0 0" rpy="${-pi/2} 0 ${-pi/2}" />
         <parent link="front_logitech" />
@@ -51,5 +52,5 @@
         </inertial>
         <visual>
-            <origin xyz="0 0 0" rpy="0 0 0" />
+            <origin xyz="0 0 0" rpy="-1.57 0 -1.57" />
             <geometry>
                 <mesh filename="file://$(find momo_description)/meshes/visual/right_logitech.STL" />
@@ -60,5 +61,5 @@
         </visual>
         <collision>
-            <origin xyz="0 0 0" rpy="0 0 0" />
+            <origin xyz="0 0 0" rpy="-1.57 0 -1.57" />
             <geometry>
                 <mesh filename="file://$(find momo_description)/meshes/visual/right_logitech.STL" />
@@ -70,9 +71,18 @@
     </gazebo>
     <joint name="right_logitech_joint" type="fixed">
-        <origin xyz="-0.00257639641022331 -0.165213293309076 0.418952968841513" rpy="-1.5707963267949 0 3.14159265358979" />
+        <!-- <origin xyz="-0.00257639641022331 -0.165213293309076 0.418952968841513" rpy="-1.5707963267949 0 3.14159265358979" /> -->
+        <origin xyz="-0.00257639641022331 -0.165213293309076 0.418952968841513" rpy="0 0 -1.57" />
         <parent link="base_link" />
         <child link="right_logitech" />
         <axis xyz="0 0 0" />
     </joint>
+    <!-- for camera plugin -->
+    <joint name="right_logitech_optical_joint" type="fixed">
+        <origin xyz="0 0 0" rpy="${-pi/2} 0 ${-pi/2}" />
+        <parent link="right_logitech" />
+        <child link="right_logitech_optical" />
+        <axis xyz="0 0 0" />
+    </joint>
+    <link name="right_logitech_optical"></link>
     <!-- BACK LOGITECH CAMERA -->
     <link name="back_logitech">
@@ -84,5 +94,5 @@
         </inertial>
         <visual>
-            <origin xyz="0 0 0" rpy="0 0 0" />
+            <origin xyz="0 0 0" rpy="-1.57 0 -1.57" />
             <geometry>
                 <mesh filename="file://$(find momo_description)/meshes/visual/back_logitech.STL" />
@@ -93,5 +103,5 @@
         </visual>
         <collision>
-            <origin xyz="0 0 0" rpy="0 0 0" />
+            <origin xyz="0 0 0" rpy="-1.57 0 -1.57" />
             <geometry>
                 <mesh filename="file://$(find momo_description)/meshes/visual/back_logitech.STL" />
@@ -103,9 +113,18 @@
     </gazebo>
     <joint name="back_logitech_joint" type="fixed">
-        <origin xyz="-0.254567242746362 0.0415958603547848 0.418952968841513" rpy="-1.5707963267949 0 1.5707963267949" />
+        <!-- <origin xyz="-0.254567242746362 0.0415958603547848 0.418952968841513" rpy="-1.5707963267949 0 1.5707963267949" /> -->
+        <origin xyz="-0.254567242746362 0.0415958603547848 0.418952968841513" rpy="0 0 3.14" />
         <parent link="base_link" />
         <child link="back_logitech" />
         <axis xyz="0 0 0" />
     </joint>
+    <!-- for camera plugin -->
+    <joint name="back_logitech_optical_joint" type="fixed">
+        <origin xyz="0 0 0" rpy="${-pi/2} 0 ${-pi/2}" />
+        <parent link="back_logitech" />
+        <child link="back_logitech_optical" />
+        <axis xyz="0 0 0" />
+    </joint>
+    <link name="back_logitech_optical"></link>
     <!-- LEFT LOGITECH CAMERA -->
     <link name="left_logitech">
@@ -117,5 +136,5 @@
         </inertial>
         <visual>
-            <origin xyz="0 0 0" rpy="0 0 0" />
+            <origin xyz="0 0 0" rpy="-1.57 0 -1.57" />
             <geometry>
                 <mesh filename="file://$(find momo_description)/meshes/visual/left_logitech.STL" />
@@ -126,5 +145,5 @@
         </visual>
         <collision>
-            <origin xyz="0 0 0" rpy="0 0 0" />
+            <origin xyz="0 0 0" rpy="-1.57 0 -1.57" />
             <geometry>
                 <mesh filename="file://$(find momo_description)/meshes/visual/left_logitech.STL" />
@@ -136,9 +155,18 @@
     </gazebo>
     <joint name="left_logitech_joint" type="fixed">
-        <origin xyz="-0.00225808908250899 0.248086706690936 0.418952968841515" rpy="-1.5707963267949 0 0" />
+        <!-- <origin xyz="-0.00225808908250899 0.248086706690936 0.418952968841515" rpy="-1.5707963267949 0 0" /> -->
+        <origin xyz="-0.00225808908250899 0.248086706690936 0.418952968841515" rpy="0 0 1.57" />
         <parent link="base_link" />
         <child link="left_logitech" />
         <axis xyz="0 0 0" />
     </joint>
+    <!-- for camera plugin -->
+    <joint name="left_logitech_optical_joint" type="fixed">
+        <origin xyz="0 0 0" rpy="-1.5707963267949 0 0" />
+        <parent link="left_logitech" />
+        <child link="left_logitech_optical" />
+        <axis xyz="0 0 0" />
+    </joint>
+    <link name="left_logitech_optical"></link>
     <!-- LIDAR -->
     <link name="lidar">
