Commit message: Update mesh file path syntax

File: momo_description/urdf/momo_core.xacro (robot description, xacro)
@@ -26,5 +26,5 @@
             <origin xyz="0 0 0" rpy="0 0 0" />
             <geometry>
-                <mesh filename="package://momo_description/meshes/visual/base_link.STL" />
+                <mesh filename="file://$(find momo_description)/meshes/visual/base_link.STL" />
             </geometry>
             <material name="">
@@ -35,5 +35,5 @@
             <origin xyz="0 0 0" rpy="0 0 0" />
             <geometry>
-                <mesh filename="package://momo_description/meshes/visual/base_link.STL" />
+                <mesh filename="file://$(find momo_description)/meshes/visual/base_link.STL" />
             </geometry>
         </collision>
@@ -50,5 +50,5 @@
             <origin xyz="0 0 0" rpy="0 0 0" />
             <geometry>
-                <mesh filename="package://momo_description/meshes/visual/front_right_wheel.STL" />
+                <mesh filename="file://$(find momo_description)/meshes/visual/front_right_wheel.STL" />
             </geometry>
             <material name="">
@@ -59,5 +59,5 @@
             <origin xyz="0 0 0" rpy="0 0 0" />
             <geometry>
-                <mesh filename="package://momo_description/meshes/visual/front_right_wheel.STL" />
+                <mesh filename="file://$(find momo_description)/meshes/visual/front_right_wheel.STL" />
             </geometry>
         </collision>
@@ -80,5 +80,5 @@
             <origin xyz="0 0 0" rpy="0 0 0" />
             <geometry>
-                <mesh filename="package://momo_description/meshes/visual/back_right_wheel.STL" />
+                <mesh filename="file://$(find momo_description)/meshes/visual/back_right_wheel.STL" />
             </geometry>
             <material name="">
@@ -89,5 +89,5 @@
             <origin xyz="0 0 0" rpy="0 0 0" />
             <geometry>
-                <mesh filename="package://momo_description/meshes/visual/back_right_wheel.STL" />
+                <mesh filename="file://$(find momo_description)/meshes/visual/back_right_wheel.STL" />
             </geometry>
         </collision>
@@ -110,5 +110,5 @@
             <origin xyz="0 0 0" rpy="0 0 0" />
             <geometry>
-                <mesh filename="package://momo_description/meshes/visual/back_left_wheel.STL" />
+                <mesh filename="file://$(find momo_description)/meshes/visual/back_left_wheel.STL" />
             </geometry>
             <material name="">
@@ -119,5 +119,5 @@
             <origin xyz="0 0 0" rpy="0 0 0" />
             <geometry>
-                <mesh filename="package://momo_description/meshes/visual/back_left_wheel.STL" />
+                <mesh filename="file://$(find momo_description)/meshes/visual/back_left_wheel.STL" />
             </geometry>
         </collision>
@@ -140,5 +140,5 @@
             <origin xyz="0 0 0" rpy="0 0 0" />
             <geometry>
-                <mesh filename="package://momo_description/meshes/visual/front_left_wheel.STL" />
+                <mesh filename="file://$(find momo_description)/meshes/visual/front_left_wheel.STL" />
             </geometry>
             <material name="">
@@ -149,5 +149,5 @@
             <origin xyz="0 0 0" rpy="0 0 0" />
             <geometry>
-                <mesh filename="package://momo_description/meshes/visual/front_left_wheel.STL" />
+                <mesh filename="file://$(find momo_description)/meshes/visual/front_left_wheel.STL" />
             </geometry>
         </collision>

File: momo_description/urdf/momo_perception_module.xacro (robot description, xacro)
@@ -12,14 +12,14 @@
             <origin xyz="0 0 0" rpy="0 0 0" />
             <geometry>
-                <mesh filename="package://momo_description/meshes/visual/front_logitech.STL" />
-            </geometry>
-            <material name="">
-                <color rgba="0.792156862745098 0.819607843137255 0.933333333333333 1" />
-            </material>
-        </visual>
-        <collision>
-            <origin xyz="0 0 0" rpy="0 0 0" />
-            <geometry>
-                <mesh filename="package://momo_description/meshes/visual/front_logitech.STL" />
+                <mesh filename="file://$(find momo_description)/meshes/visual/front_logitech.STL" />
+            </geometry>
+            <material name="">
+                <color rgba="0.792156862745098 0.819607843137255 0.933333333333333 1" />
+            </material>
+        </visual>
+        <collision>
+            <origin xyz="0 0 0" rpy="0 0 0" />
+            <geometry>
+                <mesh filename="file://$(find momo_description)/meshes/visual/front_logitech.STL" />
             </geometry>
         </collision>
@@ -42,14 +42,14 @@
             <origin xyz="0 0 0" rpy="0 0 0" />
             <geometry>
-                <mesh filename="package://momo_description/meshes/visual/right_logitech.STL" />
-            </geometry>
-            <material name="">
-                <color rgba="0.792156862745098 0.819607843137255 0.933333333333333 1" />
-            </material>
-        </visual>
-        <collision>
-            <origin xyz="0 0 0" rpy="0 0 0" />
-            <geometry>
-                <mesh filename="package://momo_description/meshes/visual/right_logitech.STL" />
+                <mesh filename="file://$(find momo_description)/meshes/visual/right_logitech.STL" />
+            </geometry>
+            <material name="">
+                <color rgba="0.792156862745098 0.819607843137255 0.933333333333333 1" />
+            </material>
+        </visual>
+        <collision>
+            <origin xyz="0 0 0" rpy="0 0 0" />
+            <geometry>
+                <mesh filename="file://$(find momo_description)/meshes/visual/right_logitech.STL" />
             </geometry>
         </collision>
@@ -72,14 +72,14 @@
             <origin xyz="0 0 0" rpy="0 0 0" />
             <geometry>
-                <mesh filename="package://momo_description/meshes/visual/back_logitech.STL" />
-            </geometry>
-            <material name="">
-                <color rgba="0.792156862745098 0.819607843137255 0.933333333333333 1" />
-            </material>
-        </visual>
-        <collision>
-            <origin xyz="0 0 0" rpy="0 0 0" />
-            <geometry>
-                <mesh filename="package://momo_description/meshes/visual/back_logitech.STL" />
+                <mesh filename="file://$(find momo_description)/meshes/visual/back_logitech.STL" />
+            </geometry>
+            <material name="">
+                <color rgba="0.792156862745098 0.819607843137255 0.933333333333333 1" />
+            </material>
+        </visual>
+        <collision>
+            <origin xyz="0 0 0" rpy="0 0 0" />
+            <geometry>
+                <mesh filename="file://$(find momo_description)/meshes/visual/back_logitech.STL" />
             </geometry>
         </collision>
@@ -102,14 +102,14 @@
             <origin xyz="0 0 0" rpy="0 0 0" />
             <geometry>
-                <mesh filename="package://momo_description/meshes/visual/left_logitech.STL" />
-            </geometry>
-            <material name="">
-                <color rgba="0.792156862745098 0.819607843137255 0.933333333333333 1" />
-            </material>
-        </visual>
-        <collision>
-            <origin xyz="0 0 0" rpy="0 0 0" />
-            <geometry>
-                <mesh filename="package://momo_description/meshes/visual/left_logitech.STL" />
+                <mesh filename="file://$(find momo_description)/meshes/visual/left_logitech.STL" />
+            </geometry>
+            <material name="">
+                <color rgba="0.792156862745098 0.819607843137255 0.933333333333333 1" />
+            </material>
+        </visual>
+        <collision>
+            <origin xyz="0 0 0" rpy="0 0 0" />
+            <geometry>
+                <mesh filename="file://$(find momo_description)/meshes/visual/left_logitech.STL" />
             </geometry>
         </collision>
@@ -132,14 +132,14 @@
             <origin xyz="0 0 0" rpy="0 0 0" />
             <geometry>
-                <mesh filename="package://momo_description/meshes/visual/lidar.STL" />
-            </geometry>
-            <material name="">
-                <color rgba="0.792156862745098 0.819607843137255 0.933333333333333 1" />
-            </material>
-        </visual>
-        <collision>
-            <origin xyz="0 0 0" rpy="0 0 0" />
-            <geometry>
-                <mesh filename="package://momo_description/meshes/visual/lidar.STL" />
+                <mesh filename="file://$(find momo_description)/meshes/visual/lidar.STL" />
+            </geometry>
+            <material name="">
+                <color rgba="0.792156862745098 0.819607843137255 0.933333333333333 1" />
+            </material>
+        </visual>
+        <collision>
+            <origin xyz="0 0 0" rpy="0 0 0" />
+            <geometry>
+                <mesh filename="file://$(find momo_description)/meshes/visual/lidar.STL" />
             </geometry>
         </collision>
@@ -162,5 +162,5 @@
             <origin xyz="0 0 0" rpy="0 0 0" />
             <geometry>
-                <mesh filename="package://momo_description/meshes/visual/realsense_t265.STL" />
+                <mesh filename="file://$(find momo_description)/meshes/visual/realsense_t265.STL" />
             </geometry>
             <material name="">
@@ -171,5 +171,5 @@
             <origin xyz="0 0 0" rpy="0 0 0" />
             <geometry>
-                <mesh filename="package://momo_description/meshes/visual/realsense_t265.STL" />
+                <mesh filename="file://$(find momo_description)/meshes/visual/realsense_t265.STL" />
             </geometry>
         </collision>
@@ -192,14 +192,14 @@
             <origin xyz="0 0 0" rpy="0 0 0" />
             <geometry>
-                <mesh filename="package://momo_description/meshes/visual/realsense_d435i.STL" />
-            </geometry>
-            <material name="">
-                <color rgba="0.792156862745098 0.819607843137255 0.933333333333333 1" />
-            </material>
-        </visual>
-        <collision>
-            <origin xyz="0 0 0" rpy="0 0 0" />
-            <geometry>
-                <mesh filename="package://momo_description/meshes/visual/realsense_d435i.STL" />
+                <mesh filename="file://$(find momo_description)/meshes/visual/realsense_d435i.STL" />
+            </geometry>
+            <material name="">
+                <color rgba="0.792156862745098 0.819607843137255 0.933333333333333 1" />
+            </material>
+        </visual>
+        <collision>
+            <origin xyz="0 0 0" rpy="0 0 0" />
+            <geometry>
+                <mesh filename="file://$(find momo_description)/meshes/visual/realsense_d435i.STL" />
             </geometry>
         </collision>
@@ -222,14 +222,14 @@
             <origin xyz="0 0 0" rpy="0 0 0" />
             <geometry>
-                <mesh filename="package://momo_description/meshes/visual/ifm_camera.STL" />
-            </geometry>
-            <material name="">
-                <color rgba="0.792156862745098 0.819607843137255 0.933333333333333 1" />
-            </material>
-        </visual>
-        <collision>
-            <origin xyz="0 0 0" rpy="0 0 0" />
-            <geometry>
-                <mesh filename="package://momo_description/meshes/visual/ifm_camera.STL" />
+                <mesh filename="file://$(find momo_description)/meshes/visual/ifm_camera.STL" />
+            </geometry>
+            <material name="">
+                <color rgba="0.792156862745098 0.819607843137255 0.933333333333333 1" />
+            </material>
+        </visual>
+        <collision>
+            <origin xyz="0 0 0" rpy="0 0 0" />
+            <geometry>
+                <mesh filename="file://$(find momo_description)/meshes/visual/ifm_camera.STL" />
             </geometry>
         </collision>

Commit message: Add gazebo colors

File: momo_description/urdf/momo_core.xacro (robot description, xacro)
@@ -39,4 +39,7 @@
         </collision>
     </link>
+    <gazebo reference="base_link">
+        <material>Gazebo/Grey</material>
+    </gazebo>
     <!-- FRONT RIGHT WHEEL -->
     <link name="front_right_wheel">
@@ -63,4 +66,7 @@
         </collision>
     </link>
+    <gazebo reference="front_right_wheel">
+        <material>Gazebo/White</material>
+    </gazebo>
     <joint name="front_right_wheel_joint" type="continuous">
         <origin xyz="0.26849 -0.318 0.059996" rpy="1.5708 0 0" />
@@ -93,4 +99,7 @@
         </collision>
     </link>
+    <gazebo reference="back_right_wheel">
+        <material>Gazebo/White</material>
+    </gazebo>
     <joint name="back_right_wheel_joint" type="continuous">
         <origin xyz="-0.27349334578749 -0.318000000000002 0.0599978846492716" rpy="1.5707963267949 0 0" />
@@ -123,4 +132,7 @@
         </collision>
     </link>
+    <gazebo reference="back_left_wheel">
+        <material>Gazebo/White</material>
+    </gazebo>
     <joint name="back_left_wheel_joint" type="continuous">
         <origin xyz="-0.273501168246142 0.318000000000003 0.0599931160727954" rpy="1.5707963267949 0 0" />
@@ -153,4 +165,7 @@
         </collision>
     </link>
+    <gazebo reference="front_left_wheel">
+        <material>Gazebo/White</material>
+    </gazebo>
     <joint name="front_left_wheel_joint" type="continuous">
         <origin xyz="0.268493050220139 0.317999999999998 0.0599993263438537" rpy="1.5707963267949 0 0" />

File: momo_description/urdf/momo_perception_module.xacro (robot description, xacro)
@@ -25,4 +25,7 @@
         </collision>
     </link>
+    <gazebo reference="front_logitech">
+        <material>Gazebo/Black</material>
+    </gazebo>
     <joint name="front_logitech_joint" type="fixed">
         <origin xyz="0.154732757253638 0.0412775530270625 0.418952968841513" rpy="-1.5707963267949 0 -1.5707963267949" />
@@ -55,4 +58,7 @@
         </collision>
     </link>
+    <gazebo reference="right_logitech">
+        <material>Gazebo/Black</material>
+    </gazebo>
     <joint name="right_logitech_joint" type="fixed">
         <origin xyz="-0.00257639641022331 -0.165213293309076 0.418952968841513" rpy="-1.5707963267949 0 3.14159265358979" />
@@ -85,4 +91,7 @@
         </collision>
     </link>
+    <gazebo reference="back_logitech">
+        <material>Gazebo/Black</material>
+    </gazebo>
     <joint name="back_logitech_joint" type="fixed">
         <origin xyz="-0.254567242746362 0.0415958603547848 0.418952968841513" rpy="-1.5707963267949 0 1.5707963267949" />
@@ -115,4 +124,7 @@
         </collision>
     </link>
+    <gazebo reference="left_logitech">
+        <material>Gazebo/Black</material>
+    </gazebo>
     <joint name="left_logitech_joint" type="fixed">
         <origin xyz="-0.00225808908250899 0.248086706690936 0.418952968841515" rpy="-1.5707963267949 0 0" />
@@ -145,4 +157,7 @@
         </collision>
     </link>
+    <gazebo reference="lidar">
+        <material>Gazebo/Grey</material>
+    </gazebo>
     <joint name="lidar_joint" type="fixed">
         <origin xyz="-0.00241706738442254 0.0414368820528667 0.478357617954853" rpy="0 0 0" />
@@ -175,4 +190,7 @@
         </collision>
     </link>
+    <gazebo reference="realsense_t265">
+        <material>Gazebo/DarkGrey</material>
+    </gazebo>
     <joint name="realsense_t265_joint" type="fixed">
         <origin xyz="0.184822757253643 0.0443427066909039 0.337457617954855" rpy="-1.5707963267949 0 -1.5707963267949" />
@@ -205,4 +223,7 @@
         </collision>
     </link>
+    <gazebo reference="realsense_d435i">
+        <material>Gazebo/DarkGrey</material>
+    </gazebo>
     <joint name="realsense_d435i_joint" type="fixed">
         <origin xyz="-0.404814742746363 0.0344707026853986 0.279039270865987" rpy="-1.5707963267949 0 1.5707963267949" />
@@ -235,4 +256,7 @@
         </collision>
     </link>
+    <gazebo reference="ifm_camera">
+        <material>Gazebo/DarkGrey</material>
+    </gazebo>
     <joint name="ifm_camera_joint" type="fixed">
         <origin xyz="0.30569 0.014587 0.26684" rpy="-1.5708 0 -1.5708" />

Commit message: Fix frame position

File: momo_description/urdf/momo_core.xacro (robot description, xacro)
@@ -51,5 +51,5 @@
         </inertial>
         <visual>
-            <origin xyz="0 0 0" rpy="0 0 0" />
+            <origin xyz="0 0 0.08" rpy="0 0 0" />
             <geometry>
                 <mesh filename="file://$(find momo_description)/meshes/visual/front_right_wheel.STL" />
@@ -60,5 +60,5 @@
         </visual>
         <collision>
-            <origin xyz="0 0 0" rpy="0 0 0" />
+            <origin xyz="0 0 0.08" rpy="0 0 0" />
             <geometry>
                 <mesh filename="file://$(find momo_description)/meshes/visual/front_right_wheel.STL" />
@@ -70,5 +70,6 @@
     </gazebo>
     <joint name="front_right_wheel_joint" type="continuous">
-        <origin xyz="0.26849 -0.318 0.059996" rpy="1.5708 0 0" />
+        <!-- <origin xyz="0.26849 -0.318 0.059996" rpy="1.5708 0 0" /> -->
+        <origin xyz="0.26849 -0.238 0.059996" rpy="1.5708 0 0" />
         <parent link="base_link" />
         <child link="front_right_wheel" />
@@ -84,5 +85,5 @@
         </inertial>
         <visual>
-            <origin xyz="0 0 0" rpy="0 0 0" />
+            <origin xyz="0 0 0.08" rpy="0 0 0" />
             <geometry>
                 <mesh filename="file://$(find momo_description)/meshes/visual/back_right_wheel.STL" />
@@ -93,5 +94,5 @@
         </visual>
         <collision>
-            <origin xyz="0 0 0" rpy="0 0 0" />
+            <origin xyz="0 0 0.08" rpy="0 0 0" />
             <geometry>
                 <mesh filename="file://$(find momo_description)/meshes/visual/back_right_wheel.STL" />
@@ -103,5 +104,6 @@
     </gazebo>
     <joint name="back_right_wheel_joint" type="continuous">
-        <origin xyz="-0.27349334578749 -0.318000000000002 0.0599978846492716" rpy="1.5707963267949 0 0" />
+        <!-- <origin xyz="-0.27349334578749 -0.318000000000002 0.0599978846492716" rpy="1.5707963267949 0 0" /> -->
+        <origin xyz="-0.27349334578749 -0.238 0.0599978846492716" rpy="1.5707963267949 0 0" />
         <parent link="base_link" />
         <child link="back_right_wheel" />

File: momo_description/urdf/momo_perception_module.xacro (robot description, xacro)
@@ -252,5 +252,5 @@
         </visual>
         <collision>
-            <origin xyz="0 0 0" rpy="0 0 0" />
+            <origin xyz="0 0 0" rpy="-1.57 0 -1.57" />
             <geometry>
                 <mesh filename="file://$(find momo_description)/meshes/visual/realsense_d435i.STL" />
