Commit message: Fix camera orientation

File: momo_description/urdf/momo_perception_module.xacro (robot description, xacro)
@@ -243,5 +243,5 @@
         </inertial>
         <visual>
-            <origin xyz="0 0 0" rpy="0 0 0" />
+            <origin xyz="0 0 0" rpy="-1.57 0 -1.57" />
             <geometry>
                 <mesh filename="file://$(find momo_description)/meshes/visual/realsense_d435i.STL" />

Commit message: Rotate lidar by 90 degrees

File: momo_description/urdf/momo_perception_module.xacro (robot description, xacro)
@@ -177,5 +177,5 @@
         </inertial>
         <visual>
-            <origin xyz="0 0 0" rpy="0 0 0" />
+            <origin xyz="0 0 0" rpy="0 0 -1.57" />
             <geometry>
                 <mesh filename="file://$(find momo_description)/meshes/visual/lidar.STL" />
@@ -186,5 +186,5 @@
         </visual>
         <collision>
-            <origin xyz="0 0 0" rpy="0 0 0" />
+            <origin xyz="0 0 0" rpy="0 0 -1.57" />
             <geometry>
                 <mesh filename="file://$(find momo_description)/meshes/visual/lidar.STL" />
