Commit message: Add dual TiM5xx lidar bringup, mocap-scenario Nav2 config, and omni teleop
- New tim_lidars.launch.py: launches both TiM5xx units (192.168.0.41 and
  192.168.1.42, the latter re-IP'd off a shared subnet) with measured
  base_link TF offsets, wired into start_up.launch.py.
- New nav2_params_mocap.yaml: no-AMCL Nav2 config for the qualisys mocap
  localization scenario, tuned MPPI/critics for the mecanum platform and
  this machine's measured compute budget.
- momo_no_master_control_mocap.launch.py: joystick strafe wiring and
  gear velocity tuning for full omnidirectional teleop driving.
- mecanum_epos4_controller.py / controller.yaml: configurable cmd_vel
  topic, staggered per-drive startup retries to absorb CAN bus init
  races.
- momo_description: removed the unused camera (logitech/realsense/ifm)
  and old lidar links from the URDF and matching xacro sources.
- mocap.rviz: fixed the 2D Goal Pose tool publishing on the unnamespaced
  /goal_pose instead of /MoMo/goal_pose.
- robotics_base: bump submodule to the strafe-support teleop branch.

File: src/momo_description/urdf/camera_plugin.xacro (robot description, xacro)
@@ -1,91 +1,3 @@
 <?xml version="1.0"?>
 <robot xmlns:xacro="https://www.ros.org/wiki/xacro">
-    <gazebo reference="front_logitech">
-        <sensor name="front_logitech_camera" type="camera">
-            <pose> 0 0 0 0 0 0 </pose>
-            <visualize>true</visualize>
-            <update_rate>10</update_rate>
-                <camera>
-                    <horizontal_fov>1.089</horizontal_fov>
-                    <image>
-                        <format>R8G8B8</format>
-                        <width>640</width>
-                        <height>480</height>
-                    </image>
-                    <clip>
-                        <near>0.05</near>
-                        <far>8.0</far>
-                    </clip>
-                </camera>
-                <plugin name="front_camera_controller" filename="libgazebo_ros_camera.so">
-                <frame_name>front_logitech_optical</frame_name>
-            </plugin>
-        </sensor>
-    </gazebo>
-    <gazebo reference="right_logitech">
-        <sensor name="right_logitech_camera" type="camera">
-            <pose> 0 0 0 0 0 0 </pose>
-            <visualize>true</visualize>
-            <update_rate>10</update_rate>
-                <camera>
-                    <horizontal_fov>1.089</horizontal_fov>
-                    <image>
-                        <format>R8G8B8</format>
-                        <width>640</width>
-                        <height>480</height>
-                    </image>
-                    <clip>
-                        <near>0.05</near>
-                        <far>8.0</far>
-                    </clip>
-                </camera>
-                <plugin name="right_camera_controller" filename="libgazebo_ros_camera.so">
-                <frame_name>right_logitech_optical</frame_name>
-            </plugin>
-        </sensor>
-    </gazebo>
-    <gazebo reference="back_logitech">
-        <sensor name="back_logitech_camera" type="camera">
-            <pose> 0 0 0 0 0 0 </pose>
-            <visualize>true</visualize>
-            <update_rate>10</update_rate>
-                <camera>
-                    <horizontal_fov>1.089</horizontal_fov>
-                    <image>
-                        <format>R8G8B8</format>
-                        <width>640</width>
-                        <height>480</height>
-                    </image>
-                    <clip>
-                        <near>0.05</near>
-                        <far>8.0</far>
-                    </clip>
-                </camera>
-                <plugin name="back_camera_controller" filename="libgazebo_ros_camera.so">
-                <frame_name>back_logitech_optical</frame_name>
-            </plugin>
-        </sensor>
-    </gazebo>
-    <gazebo reference="left_logitech">
-        <sensor name="left_logitech_camera" type="camera">
-            <pose> 0 0 0 0 0 0 </pose>
-            <visualize>true</visualize>
-            <update_rate>10</update_rate>
-                <camera>
-                    <horizontal_fov>1.089</horizontal_fov>
-                    <image>
-                        <format>R8G8B8</format>
-                        <width>640</width>
-                        <height>480</height>
-                    </image>
-                    <clip>
-                        <near>0.05</near>
-                        <far>8.0</far>
-                    </clip>
-                </camera>
-                <plugin name="left_camera_controller" filename="libgazebo_ros_camera.so">
-                <frame_name>left_logitech_optical</frame_name>
-            </plugin>
-        </sensor>
-    </gazebo>
 </robot>

File: src/momo_description/urdf/depth_camera_plugin.xacro (robot description, xacro)
@@ -1,27 +1,3 @@
 <?xml version="1.0"?>
 <robot xmlns:xacro="https://www.ros.org/wiki/xacro">
-    <gazebo reference="realsense_d435i">  <!-- reference is the link name in the urdf -->
-        <sensor name="realsense_d435i_camera" type="depth"> <!-- name is the link_name_camera -->
-            <pose> 0 0 0 0 0 0 </pose>
-            <visualize>true</visualize>
-            <update_rate>10</update_rate>
-                <camera>
-                    <horizontal_fov>1.089</horizontal_fov>
-                    <image>
-                        <format>B8G8R8</format>
-                        <width>640</width>
-                        <height>480</height>
-                    </image>
-                    <clip>
-                        <near>0.05</near>
-                        <far>8.0</far>
-                    </clip>
-                </camera>
-                <plugin name="realsense_d435i_controller" filename="libgazebo_ros_camera.so"> <!-- name refers to the node name-->
-                <frame_name>realsense_d435i_optical</frame_name>
-                <min_depth>0.1</min_depth>
-                <max_depth>100.0</max_depth>
-            </plugin>
-        </sensor>
-    </gazebo>
 </robot>

File: src/momo_description/urdf/lidar_plugin.xacro (robot description, xacro)
@@ -1,30 +1,3 @@
 <?xml version="1.0"?>
 <robot xmlns:xacro="https://www.ros.org/wiki/xacro">
-    <gazebo reference="lidar">
-        <sensor name="laser" type="ray">
-            <pose> 0 0 0 0 0 0 </pose>
-            <visualize>false</visualize>
-            <update_rate>10</update_rate>
-            <ray>
-                <scan>
-                    <horizontal>
-                        <samples>360</samples>
-                        <min_angle>-3.14</min_angle>
-                        <max_angle>3.14</max_angle>
-                    </horizontal>
-                </scan>
-                <range>
-                    <min>0.3</min>
-                    <max>12</max>
-                </range>
-            </ray>
-            <plugin name="laser_controller" filename="libgazebo_ros_ray_sensor.so">
-                <ros>
-                    <argument>~/out:=scan</argument>
-                </ros>
-                <output_type>sensor_msgs/LaserScan</output_type>
-                <frame_name>lidar</frame_name>
-            </plugin>
-        </sensor>
-    </gazebo>
 </robot>

File: src/momo_description/urdf/momo_description.urdf (robot description, URDF)
Before this commit: robot momo_description, 14 links, 13 joints
Links:
- removed link back_logitech
- removed link front_logitech
- removed link ifm_camera
- removed link left_logitech
- removed link lidar
- removed link realsense_d435i
- removed link realsense_t265
- removed link right_logitech
Joints:
- removed joint back_logitech_joint
- removed joint front_logitech_joint
- removed joint ifm_camera_joint
- removed joint left_logitech_joint
- removed joint lidar_joint
- removed joint realsense_d435i_joint
- removed joint realsense_t265_joint
- removed joint right_logitech_joint

File: src/momo_description/urdf/momo_perception_module.xacro (robot description, xacro)
@@ -1,310 +1,3 @@
 <?xml version="1.0"?>
 <robot xmlns:xacro="http://www.ros.org/wiki/xacro">
-    <!-- FRONT LOGITECH CAMERA -->
-    <link name="front_logitech">
-        <inertial>
-            <origin xyz="-0.000100619366527013 0.00868433169256161 -0.0237131147679362" rpy="0 0 0" />
-            <mass value="0.0873967458266508" />
-            <inertia ixx="3.99321306212914E-05" ixy="-2.39081067841113E-08" ixz="-7.19738531428668E-08"
-                    iyy="6.41203019340331E-05" iyz="1.1807193889875E-05" izz="5.08960858757451E-05" />
-        </inertial>
-        <visual>
-            <origin xyz="0 0 0" rpy="-1.57 0 -1.57" />
-            <geometry>
-                <mesh filename="file://$(find momo_description)/meshes/visual/front_logitech.STL" />
-            </geometry>
-            <material name="">
-                <color rgba="0.792156862745098 0.819607843137255 0.933333333333333 1" />
-            </material>
-        </visual>
-        <collision>
-            <origin xyz="0 0 0" rpy="-1.57 0 -1.57" />
-            <geometry>
-                <mesh filename="file://$(find momo_description)/meshes/visual/front_logitech.STL" />
-            </geometry>
-        </collision>
-    </link>
-    <gazebo reference="front_logitech">
-        <material>Gazebo/Black</material>
-    </gazebo>
-    <joint name="front_logitech_joint" type="fixed">
-        <origin xyz="0.154732757253638 0.0412775530270625 0.418952968841513" rpy="0 0 0" />
-        <parent link="base_link" />
-        <child link="front_logitech" />
-        <axis xyz="0 0 0" />
-    </joint>
-    <!-- for camera plugin -->
-    <joint name="front_logitech_optical_joint" type="fixed"> <!-- link_name_optical_joint -->
-        <origin xyz="0 0 0" rpy="${-pi/2} 0 ${-pi/2}" />     <!-- this line always stays the same -->
-        <parent link="front_logitech" />                     <!-- link_name -->
-        <child link="front_logitech_optical" />              <!-- link_name_optical -->
-        <axis xyz="0 0 0" />
-    </joint>
-    <link name="front_logitech_optical"></link>              <!-- link_name_optical -->
-    <!-- RIGHT LOGITECH CAMERA -->
-    <link name="right_logitech">
-        <inertial>
-            <origin xyz="-0.000100619366454141 0.00868433169256244 -0.0237131147679361" rpy="0 0 0" />
-            <mass value="0.0873967458266508" />
-            <inertia ixx="3.99321306212963E-05" ixy="-2.39081065814224E-08" ixz="-7.19738530417854E-08"
-                    iyy="6.41203019340384E-05" iyz="1.18071938898757E-05" izz="5.08960858757447E-05" />
-        </inertial>
-        <visual>
-            <origin xyz="0 0 0" rpy="-1.57 0 -1.57" />
-            <geometry>
-                <mesh filename="file://$(find momo_description)/meshes/visual/right_logitech.STL" />
-            </geometry>
-            <material name="">
-                <color rgba="0.792156862745098 0.819607843137255 0.933333333333333 1" />
-            </material>
-        </visual>
-        <collision>
-            <origin xyz="0 0 0" rpy="-1.57 0 -1.57" />
-            <geometry>
-                <mesh filename="file://$(find momo_description)/meshes/visual/right_logitech.STL" />
-            </geometry>
-        </collision>
-    </link>
-    <gazebo reference="right_logitech">
-        <material>Gazebo/Black</material>
-    </gazebo>
-    <joint name="right_logitech_joint" type="fixed">
-        <!-- <origin xyz="-0.00257639641022331 -0.165213293309076 0.418952968841513" rpy="-1.5707963267949 0 3.14159265358979" /> -->
-        <origin xyz="-0.00257639641022331 -0.165213293309076 0.418952968841513" rpy="0 0 -1.57" />
-        <parent link="base_link" />
-        <child link="right_logitech" />
-        <axis xyz="0 0 0" />
-    </joint>
-    <!-- for camera plugin -->
-    <joint name="right_logitech_optical_joint" type="fixed">
-        <origin xyz="0 0 0" rpy="${-pi/2} 0 ${-pi/2}" />
-        <parent link="right_logitech" />
-        <child link="right_logitech_optical" />
-        <axis xyz="0 0 0" />
-    </joint>
-    <link name="right_logitech_optical"></link>
-    <!-- BACK LOGITECH CAMERA -->
-    <link name="back_logitech">
-        <inertial>
-            <origin xyz="-0.000100619366527027 0.00868433169256172 -0.0237131147679362" rpy="0 0 0" />
-            <mass value="0.0873967458266511" />
-            <inertia ixx="3.99321306212934E-05" ixy="-2.39081067841115E-08" ixz="-7.19738531417099E-08"
-                    iyy="6.41203019340351E-05" iyz="1.18071938898751E-05" izz="5.08960858757451E-05" />
-        </inertial>
-        <visual>
-            <origin xyz="0 0 0" rpy="-1.57 0 -1.57" />
-            <geometry>
-                <mesh filename="file://$(find momo_description)/meshes/visual/back_logitech.STL" />
-            </geometry>
-            <material name="">
-                <color rgba="0.792156862745098 0.819607843137255 0.933333333333333 1" />
-            </material>
-        </visual>
-        <collision>
-            <origin xyz="0 0 0" rpy="-1.57 0 -1.57" />
-            <geometry>
-                <mesh filename="file://$(find momo_description)/meshes/visual/back_logitech.STL" />
-            </geometry>
-        </collision>
-    </link>
-    <gazebo reference="back_logitech">
-        <material>Gazebo/Black</material>
-    </gazebo>
-    <joint name="back_logitech_joint" type="fixed">
-        <!-- <origin xyz="-0.254567242746362 0.0415958603547848 0.418952968841513" rpy="-1.5707963267949 0 1.5707963267949" /> -->
-        <origin xyz="-0.254567242746362 0.0415958603547848 0.418952968841513" rpy="0 0 3.14" />
-        <parent link="base_link" />
-        <child link="back_logitech" />
-        <axis xyz="0 0 0" />
-    </joint>
-    <!-- for camera plugin -->
-    <joint name="back_logitech_optical_joint" type="fixed">
-        <origin xyz="0 0 0" rpy="${-pi/2} 0 ${-pi/2}" />
-        <parent link="back_logitech" />
-        <child link="back_logitech_optical" />
-        <axis xyz="0 0 0" />
-    </joint>
-    <link name="back_logitech_optical"></link>
-    <!-- LEFT LOGITECH CAMERA -->
-    <link name="left_logitech">
-        <inertial>
-            <origin xyz="-0.000100619366454391 0.0086843316925625 -0.0237131147679363" rpy="0 0 0" />
-            <mass value="0.0873967458266511" />
-            <inertia ixx="3.99321306212903E-05" ixy="-2.39081065815171E-08" ixz="-7.19738530421334E-08"
-                    iyy="6.41203019340324E-05" iyz="1.18071938898756E-05" izz="5.08960858757447E-05" />
-        </inertial>
-        <visual>
-            <origin xyz="0 0 0" rpy="-1.57 0 -1.57" />
-            <geometry>
-                <mesh filename="file://$(find momo_description)/meshes/visual/left_logitech.STL" />
-            </geometry>
-            <material name="">
-                <color rgba="0.792156862745098 0.819607843137255 0.933333333333333 1" />
-            </material>
-        </visual>
-        <collision>
-            <origin xyz="0 0 0" rpy="-1.57 0 -1.57" />
-            <geometry>
-                <mesh filename="file://$(find momo_description)/meshes/visual/left_logitech.STL" />
-            </geometry>
-        </collision>
-    </link>
-    <gazebo reference="left_logitech">
-        <material>Gazebo/Black</material>
-    </gazebo>
-    <joint name="left_logitech_joint" type="fixed">
-        <!-- <origin xyz="-0.00225808908250899 0.248086706690936 0.418952968841515" rpy="-1.5707963267949 0 0" /> -->
-        <origin xyz="-0.00225808908250899 0.248086706690936 0.418952968841515" rpy="0 0 1.57" />
-        <parent link="base_link" />
-        <child link="left_logitech" />
-        <axis xyz="0 0 0" />
-    </joint>
-    <!-- for camera plugin -->
-    <joint name="left_logitech_optical_joint" type="fixed">
-        <origin xyz="0 0 0" rpy="${-pi/2} 0 ${-pi/2}" />
-        <parent link="left_logitech" />
-        <child link="left_logitech_optical" />
-        <axis xyz="0 0 0" />
-    </joint>
-    <link name="left_logitech_optical"></link>
-    <!-- LIDAR -->
-    <link name="lidar">
-        <inertial>
-            <origin xyz="-3.2878099134187E-06 -0.000102126009981357 -0.00210332117212092" rpy="0 0 0" />
-            <mass value="0.605610123538718" />
-            <inertia ixx="0.000670924573306349" ixy="-5.82638316928472E-12" ixz="-6.67755541756334E-08"
-                    iyy="0.000667040687285356" iyz="-1.81285167753324E-06" izz="0.000804073760064738" />
-        </inertial>
-        <visual>
-            <origin xyz="0 0 0" rpy="0 0 -1.57" />
-            <geometry>
-                <mesh filename="file://$(find momo_description)/meshes/visual/lidar.STL" />
-            </geometry>
-            <material name="">
-                <color rgba="0.792156862745098 0.819607843137255 0.933333333333333 1" />
-            </material>
-        </visual>
-        <collision>
-            <origin xyz="0 0 0" rpy="0 0 -1.57" />
-            <geometry>
-                <mesh filename="file://$(find momo_description)/meshes/visual/lidar.STL" />
-            </geometry>
-        </collision>
-    </link>
-    <gazebo reference="lidar">
-        <material>Gazebo/Grey</material>
-    </gazebo>
-    <joint name="lidar_joint" type="fixed">
-        <origin xyz="-0.00241706738442254 0.0414368820528667 0.478357617954853" rpy="0 0 0" />
-        <parent link="base_link" />
-        <child link="lidar" />
-        <axis xyz="0 0 0" />
-    </joint>
-    <!-- REALSENSE T265 -->
-    <link name="realsense_t265">
-        <inertial>
-            <origin xyz="0.000129462657322346 -1.57181139381901E-07 -0.00601066388944044" rpy="0 0 0" />
-            <mass value="0.0311240910368595" />
-            <inertia ixx="1.83337825677375E-06" ixy="-2.85176636894001E-10" ixz="-7.81020859395691E-09"
-                    iyy="2.96344209179022E-05" iyz="1.3923224154143E-11" izz="3.06979172999491E-05" />
-        </inertial>
-        <visual>
-            <origin xyz="0 0 0" rpy="0 0 0" />
-            <geometry>
-                <mesh filename="file://$(find momo_description)/meshes/visual/realsense_t265.STL" />
-            </geometry>
-            <material name="">
-                <color rgba="0.627450980392157 0.627450980392157 0.627450980392157 1" />
-            </material>
-        </visual>
-        <collision>
-            <origin xyz="0 0 0" rpy="0 0 0" />
-            <geometry>
-                <mesh filename="file://$(find momo_description)/meshes/visual/realsense_t265.STL" />
-            </geometry>
-        </collision>
-    </link>
-    <gazebo reference="realsense_t265">
-        <material>Gazebo/DarkGrey</material>
-    </gazebo>
-    <joint name="realsense_t265_joint" type="fixed">
-        <origin xyz="0.184822757253643 0.0443427066909039 0.337457617954855" rpy="-1.5707963267949 0 -1.5707963267949" />
-        <parent link="base_link" />
-        <child link="realsense_t265" />
-        <axis xyz="0 0 0" />
-    </joint>
-    <!-- REALSENSE D435I -->
-    <link name="realsense_d435i">
-        <inertial>
-            <origin xyz="-0.000995206394463141 2.7881471328095E-05 -0.0125659497249071" rpy="0 0 0" />
-            <mass value="0.0457663452618203" />
-            <inertia ixx="4.14998076783152E-06" ixy="-1.50844318927118E-09" ixz="-4.10538526085445E-07"
-                    iyy="2.78843613995507E-05" iyz="-7.38862868090377E-09" izz="2.75878432161684E-05" />
-        </inertial>
-        <visual>
-            <origin xyz="0 0 0" rpy="-1.57 0 -1.57" />
-            <geometry>
-                <mesh filename="file://$(find momo_description)/meshes/visual/realsense_d435i.STL" />
-            </geometry>
-            <material name="">
-                <color rgba="0.792156862745098 0.819607843137255 0.933333333333333 1" />
-            </material>
-        </visual>
-        <collision>
-            <origin xyz="0 0 0" rpy="-1.57 0 -1.57" />
-            <geometry>
-                <mesh filename="file://$(find momo_description)/meshes/visual/realsense_d435i.STL" />
-            </geometry>
-        </collision>
-    </link>
-    <gazebo reference="realsense_d435i">
-        <material>Gazebo/DarkGrey</material>
-    </gazebo>
-    <joint name="realsense_d435i_joint" type="fixed">
-        <origin xyz="-0.404814742746363 0.0344707026853986 0.279039270865987" rpy="0 0 3.14" />
-        <parent link="base_link" />
-        <child link="realsense_d435i" />
-        <axis xyz="0 0 0" />
-    </joint>
-    <!-- for depth camera plugin -->
-    <joint name="realsense_d435i_optical_joint" type="fixed">
-        <origin xyz="0 0 0" rpy="${-pi/2} 0 ${-pi/2}" />
-        <parent link="realsense_d435i" />
-        <child link="realsense_d435i_optical" />
-        <axis xyz="0 0 0" />
-    </joint>
-    <link name="realsense_d435i_optical"></link>
-    <!-- IFM CAMERA -->
-    <link name="ifm_camera">
-        <inertial>
-            <origin xyz="-0.0227481615945184 3.06773217939593E-11 -0.0127352941193509" rpy="0 0 0" />
-            <mass value="0.0711675681323896" />
-            <inertia ixx="9.48525117222579E-06" ixy="1.49142424517477E-13" ixz="-6.00059122328344E-08"
-                    iyy="5.23565081343951E-05" iyz="-8.51988151121233E-15" izz="5.41536530687776E-05" />
-        </inertial>
-        <visual>
-            <origin xyz="0 0 0" rpy="0 0 0" />
-            <geometry>
-                <mesh filename="file://$(find momo_description)/meshes/visual/ifm_camera.STL" />
-            </geometry>
-            <material name="">
-                <color rgba="0.792156862745098 0.819607843137255 0.933333333333333 1" />
-            </material>
-        </visual>
-        <collision>
-            <origin xyz="0 0 0" rpy="0 0 0" />
-            <geometry>
-                <mesh filename="file://$(find momo_description)/meshes/visual/ifm_camera.STL" />
-            </geometry>
-        </collision>
-    </link>
-    <gazebo reference="ifm_camera">
-        <material>Gazebo/DarkGrey</material>
-    </gazebo>
-    <joint name="ifm_camera_joint" type="fixed">
-        <origin xyz="0.30569 0.014587 0.26684" rpy="-1.5708 0 -1.5708" />
-        <parent link="base_link" />
-        <child link="ifm_camera" />
-        <axis xyz="0 0 0" />
-    </joint>
 </robot>
